Commit message: feat: perception classification + ReAct reasoning + hardware commissioning prep
A2: Shape classification (PCA eigenvalue ratios) + color extraction (HSV from RGB pointcloud)
A3: Human-readable detection descriptions for LLM agent (query_perception_tool)
B1: Enhanced ReAct system prompt with multi-step reasoning, safety rules, tool chaining
Hardware gate: checklist approved for commissioning

- scene_processor: _classify_shape(), _dominant_color_name(), _read_xyz_rgb()
- query_perception_tool: _format_detection(), _format_detections_from_ros()
- react_planner: enriched perception output, structured prompt sections
- All 409 tests pass (40 gp4_perception + 369 llm_gateway)
- Camera D435i config, calibration launch, URDF updates
- HMI, safety, motion_core, hw_adapter refactoring from W1-W8

File: src/gp4_station/urdf/gp4_on_station.urdf.xacro (robot description, xacro)
@@ -31,3 +31,67 @@
   </joint>
   <xacro:motoman_gp4 prefix="" />
+  <!-- ============================================================
+       D435i Camera — eye-to-hand, upper-left front corner of station
+       ============================================================
+       Position is NOMINAL from CAD. The actual camera-to-robot
+       transform comes from hand-eye calibration (extrinsics.yaml).
+       This link exists for:
+         1. RViz visualisation of camera position
+         2. MoveIt collision avoidance (camera body as collision box)
+         3. Approximate TF seed before calibration is run
+       Camera orientation convention (RealSense optical frame):
+         Z = forward (optical axis), X = right, Y = down
+       Mount description (operator perspective, facing station front):
+         - Upper-left corner of station aluminium frame
+         - Pitch down ~40° towards workspace centre
+         - Yaw inward ~20° towards positive-Y in base_link
+       ============================================================ -->
+  <!-- Camera mount bracket (fixed to station frame) -->
+  <link name="camera_mount_link" />
+  <joint name="station_to_camera_mount" type="fixed">
+    <parent link="station_link" />
+    <child link="camera_mount_link" />
+    <!-- TBD: operator must measure and update after physical mounting.
+         Current values are estimates from CAD images (station frame). -->
+    <origin xyz="-0.30 -0.10 0.15" rpy="0 0 0" />
+  </joint>
+  <!-- Camera body link with collision box for MoveIt planning -->
+  <link name="camera_link">
+    <visual>
+      <origin xyz="0 0 0" rpy="0 0 0" />
+      <geometry>
+        <!-- D435i physical dimensions: 90mm × 25mm × 25mm -->
+        <box size="0.090 0.025 0.025" />
+      </geometry>
+      <material name="camera_black">
+        <color rgba="0.15 0.15 0.15 1.0" />
+      </material>
+    </visual>
+    <collision>
+      <origin xyz="0 0 0" rpy="0 0 0" />
+      <geometry>
+        <!-- Slightly inflated for collision safety margin -->
+        <box size="0.100 0.035 0.035" />
+      </geometry>
+    </collision>
+  </link>
+  <joint name="camera_mount_to_camera" type="fixed">
+    <parent link="camera_mount_link" />
+    <child link="camera_link" />
+    <!-- Pitch ~40° down (0.698 rad), yaw ~20° inward (0.349 rad).
+         TBD: operator must verify orientation after mounting. -->
+    <origin xyz="0 0 0" rpy="0 0.698 0.349" />
+  </joint>
+  <!-- Camera optical frame (follows ROS/OpenCV convention: Z-forward, X-right, Y-down).
+       The realsense2_camera node publishes its own camera_color_optical_frame TF,
+       but this link lets the URDF TF tree stay connected even without the camera running.
+       After hand-eye calibration, the TFPublisher node overrides base_link → camera_color_optical_frame
+       with the precise calibrated transform from extrinsics.yaml. -->
+  <link name="camera_color_optical_frame_nominal" />
+  <joint name="camera_to_optical_nominal" type="fixed">
+    <parent link="camera_link" />
+    <child link="camera_color_optical_frame_nominal" />
+    <!-- ROS convention → optical frame: rotate -90° around Z, then -90° around X -->
+    <origin xyz="0 0 0" rpy="-1.5708 0 -1.5708" />
+  </joint>
 </robot>

Commit message: feat: optimize GP4 HMI interface, implement observability console, and refine camera calibration

File: src/gp4_station/urdf/gp4_on_station.urdf.xacro (robot description, xacro)
@@ -54,5 +54,5 @@
     <!-- TBD: operator must measure and update after physical mounting.
          Current values are estimates from CAD images (station frame). -->
-    <origin xyz="-0.30 -0.10 0.15" rpy="0 0 0" />
+    <origin xyz="-1.093 -0.504 0.636" rpy="0 0 0" />
   </joint>
   <!-- Camera body link with collision box for MoveIt planning -->

Commit message: ws-deep-rebuild: perception uplift, react-vision composite, motion_core guards, llm_gateway refactor, hmi fixes
- gp4_perception: query_perception_tool rewrite (+729 lines), scene_processor
  expansion, calibration updates, new detection_visualizer, config overhauls
- llm_gateway: react_planner rewrite, semantic_ir_contract expansion,
  llm_gateway_node refactor, new test_direct_review_regex
- motion_core: trajectory_validator header/impl, joint_position_guard hardening,
  move_rel_validator updates, quality_gate wiring, primitive_router_dispatch
  updates, motion_core_node YAML loading, new test_trajectory_validator
- hmi: backend contract/model/sequence/submission/view changes, frontend
  GP4HMI/SystemLog/derive/types updates, system-log CSS
- safety: safety_rules.yaml operational limits, execution_gate updates,
  station_geometry_policy_sync test updates
- gp4_station: URDF updates
- gp4_bringup: launch test fix
- tools: generate_aruco_board, runtime_console updates, new
  test_runtime_console.py
- docs: HMI interfaces, perception runbook, react-vision spec

File: src/gp4_station/urdf/gp4_on_station.urdf.xacro (robot description, xacro)
@@ -32,8 +32,9 @@
   <xacro:motoman_gp4 prefix="" />
   <!-- ============================================================
-       D435i Camera — eye-to-hand, upper-left front corner of station
+       D435i Camera — eye-to-hand, front-center above robot base
        ============================================================
-       Position is NOMINAL from CAD. The actual camera-to-robot
-       transform comes from hand-eye calibration (extrinsics.yaml).
+       Position is NOMINAL from physical measurement (scale 0.25).
+       The actual camera-to-robot transform comes from hand-eye
+       calibration (extrinsics.yaml).
        This link exists for:
          1. RViz visualisation of camera position
@@ -43,16 +44,15 @@
          Z = forward (optical axis), X = right, Y = down
        Mount description (operator perspective, facing station front):
-         - Upper-left corner of station aluminium frame
-         - Pitch down ~40° towards workspace centre
-         - Yaw inward ~20° towards positive-Y in base_link
+         - Front of robot (facing direction at HOME pose), centred on base_link Y axis (X ≈ 0)
+         - Diagonal distance from base origin to camera: ~1025 mm
+         - Horizontal/vertical leg of the diagonal: ~724 mm each
+         - Pitch down ~45° towards base origin
        ============================================================ -->
-  <!-- Camera mount bracket (fixed to station frame) -->
+  <!-- Camera mount bracket (fixed directly to robot base for clarity) -->
   <link name="camera_mount_link" />
-  <joint name="station_to_camera_mount" type="fixed">
-    <parent link="station_link" />
+  <joint name="base_to_camera_mount" type="fixed">
+    <parent link="base_link" />
     <child link="camera_mount_link" />
-    <!-- TBD: operator must measure and update after physical mounting.
-         Current values are estimates from CAD images (station frame). -->
-    <origin xyz="-1.093 -0.504 0.636" rpy="0 0 0" />
+    <origin xyz="0.0 0.724 0.726" rpy="0 0 0" />
   </joint>
   <!-- Camera body link with collision box for MoveIt planning -->
@@ -79,19 +79,16 @@
     <parent link="camera_mount_link" />
     <child link="camera_link" />
-    <!-- Pitch ~40° down (0.698 rad), yaw ~20° inward (0.349 rad).
-         TBD: operator must verify orientation after mounting. -->
-    <origin xyz="0 0 0" rpy="0 0.698 0.349" />
+    <!-- Optical frame directly: Z forward toward robot base, X right, Y down -->
+    <origin xyz="0 0 0" rpy="2.356 0 3.1416" />
   </joint>
-  <!-- Camera optical frame (follows ROS/OpenCV convention: Z-forward, X-right, Y-down).
-       The realsense2_camera node publishes its own camera_color_optical_frame TF,
-       but this link lets the URDF TF tree stay connected even without the camera running.
-       After hand-eye calibration, the TFPublisher node overrides base_link → camera_color_optical_frame
-       with the precise calibrated transform from extrinsics.yaml. -->
+  <!-- Camera optical frame — same as camera_link for visual clarity.
+       The realsense2_camera node publishes its own camera_color_optical_frame TF.
+       This link keeps the URDF TF tree connected when the camera is offline. -->
   <link name="camera_color_optical_frame_nominal" />
   <joint name="camera_to_optical_nominal" type="fixed">
     <parent link="camera_link" />
     <child link="camera_color_optical_frame_nominal" />
-    <!-- ROS convention → optical frame: rotate -90° around Z, then -90° around X -->
-    <origin xyz="0 0 0" rpy="-1.5708 0 -1.5708" />
+    <!-- Identity: camera_link already uses optical convention in this setup -->
+    <origin xyz="0 0 0" rpy="0 0 0" />
   </joint>
 </robot>
