Commit message: refactor: complete workspace-wide refactor across all active packages
Consolidates remaining changes from the super-fix refactor branch:
- HMI: command ingress contracts, jog dispatch, supervisor service splits
- interfaces: DispatchTrajectory action updates, package metadata
- motion_core: move_rel_validator, planning_scene_manager, seed_manager,
  quality_gate, wrist_flip_guard improvements
- hw_adapter: trajectory_executor, robot_status_monitor, node updates
- llm_gateway: goal_mapper, normalizer, prompt_builder, semantic_validator,
  schema alignment
- safety: execution_gate, command_validator, safety_rules config
- gp4_bringup: launch files, scene_objects, CMake/package updates
- gp4_moveit_config: kinematics, URDF xacro, servo config
- jog_pendant: servo_bridge_node, experimental launch
- Tests updated across all packages

File: src/gp4_moveit_config/config/motoman_gp4.urdf.xacro (robot description, xacro)
@@ -14,4 +14,25 @@
     <!-- Import ros2_control xacro -->
     <xacro:include filename="motoman_gp4.ros2_control.xacro" />
+    <!--
+      Station visual is embedded in MoveIt robot_description so gp4_bringup
+      always shows the real cell model in RViz.
+      Collision authority stays in gp4_bringup/config/scene_objects.yaml.
+    -->
+    <link name="station_visual_link">
+      <visual>
+        <origin xyz="0 0 0" rpy="0 0 0" />
+        <geometry>
+          <mesh filename="package://gp4_station/meshes/station3.stl" scale="0.001 0.001 0.001" />
+        </geometry>
+        <material name="station_grey">
+          <color rgba="0.35 0.35 0.35 1.0" />
+        </material>
+      </visual>
+    </link>
+    <joint name="base_to_station_visual" type="fixed">
+      <parent link="base_link" />
+      <child link="station_visual_link" />
+      <origin xyz="0 0 0" rpy="0 0 ${pi}" />
+    </joint>
     <!-- Gọi macro với tham số thật/giả -->
     <xacro:motoman_gp4_ros2_control

Commit message: feat: update HMI components, LLM gateway logic and robot configurations

File: src/gp4_moveit_config/config/motoman_gp4.urdf.xacro (robot description, xacro)
@@ -12,4 +12,11 @@
     <!-- Import motoman_gp4 urdf file -->
     <xacro:include filename="$(find motoman_gp4_support)/urdf/gp4.urdf" />
+    <!-- TCP Link configuration: 11cm (0.11m) from tool0 -->
+    <link name="tcp_link" />
+    <joint name="tool0_to_tcp" type="fixed">
+      <parent link="tool0" />
+      <child link="tcp_link" />
+      <origin xyz="0 0 0.11" rpy="0 0 0" />
+    </joint>
     <!-- Import ros2_control xacro -->
     <xacro:include filename="motoman_gp4.ros2_control.xacro" />

Commit message: Calibrate robot perception extrinsics, calculate jerk, fix UI TCP values

File: src/gp4_moveit_config/config/motoman_gp4.urdf.xacro (robot description, xacro)
@@ -17,5 +17,5 @@
       <parent link="tool0" />
       <child link="tcp_link" />
-      <origin xyz="0 0 0.11" rpy="0 0 0" />
+      <origin xyz="0.05 0 0.115" rpy="0 0 0" />
     </joint>
     <!-- Import ros2_control xacro -->
